File: pcb/TM4C1294/TM4C1294.sch (KiCad schematic (older format))
At the start: 38 parts, among them J1 EK-TM4C1294, Q1 PN2222A, Q2 PN2222A, Q3 PN2222A, Q4 PN2222A, T1 Keypad4x4, U1 CA56-12CGKWA

Commit message: Version 1.0
Other:
- note added: "Display 7 segmentos de 4 digitos"
- note added: "EK-TM4C1294XL"
- note added: "LCD Nokia 5110\n"
- note added: "Leds de salida"
- note added: "Teclado matricial 4x4"
- moved on the sheet: BAR1, FID1, FID2, FID3, H1, H2, H3, H4, J1A, J1B, J1C, J1D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

Commit message: Version 1.0
Parts:
- removed T1: Keypad4x4, EK-TM4C1294:Keypad, symbol EK-TM4C1294:Keypad4x4
- added T?: Keypad4x4, EK-TM4C1294:Keypad, symbol EK-TM4C1294:Keypad4x4
Connections:
- net PC4: now also T?.5
- net PC5: now also T?.6
- net PC6: now also T?.6
- net PC7: now also T?.7
- net PE0: now also T?.1
- net PE1: now also T?.2
- net PE2: now also T?.3
- net PE3: now also T?.4
Changed lines of the file:
@@
-$EndComp
-$Comp
-L EK-TM4C1294:Keypad4x4 T1
-U 1 1 614CEC02
-P 6300 1600
-F 0 "T1" H 6850 2300 50  0000 L CNN
-F 1 "Keypad4x4" H 6350 2300 50  0000 L CNN
-F 2 "EK-TM4C1294:Keypad" H 6300 1300 50  0001 C CNN
-F 3 "https://cdn.sparkfun.com/assets/f/f/a/5/0/DS-16038.pdf" H 6300 1300 50  0001 C CNN
-	1    6300 1600
-	1    0    0    -1
 $EndComp
 $Comp
@@
 Wire Notes Line
 	750  700  750  6800
+$Comp
+L EK-TM4C1294:Keypad4x4 T?
+U 1 1 614E30AE
+P 6300 1600
+F 0 "T?" H 6978 1913 50  0000 L CNN
+F 1 "Keypad4x4" H 6978 1822 50  0000 L CNN
+F 2 "EK-TM4C1294:Keypad" H 6300 1300 50  0001 C CNN
+F 3 "https://cdn.sparkfun.com/assets/f/f/a/5/0/DS-16038.pdf" H 6300 1300 50  0001 C CNN
+	1    6300 1600
+	1    0    0    -1
+$EndComp
 $EndSCHEMATC
